File: KicadJE_RIAA_RevA/KicadJE_RIAA.kicad_pcb (KiCad board)
At the start: 2 copper layers, 100 x 100 mm, 202 parts, among them J201 In_Accent, J202 In Gate, J203 Out Tom, J301 PJRAS2X2S01AUX, J302 Conn_01x03, P201 Doepfer_Power_10pin, Q201 MMBT2222A, Q202 MMBT2222A, Q203 MMBT2222A, Q204 MMBT2222A, Q205 MMBT2907A, Q206 MMBT2222A, Q207 MMBT2222A, SW201 Con/Tom, U201 TL072, U202 TL072, U203 TL072, U301 TL072, U302 TL072, U303 TL072

Commit message: Update KicadJE_RIAA.kicad_pcb
Parts:
- removed C201, C202, C203, C204: 100n, Capacitor_SMD:C_0805_2012Metric_Pad1.15x1.40mm_HandSolder
- removed C205: 39n, Capacitor_SMD:C_0805_2012Metric_Pad1.15x1.40mm_HandSolder
- removed C206: 1u, Capacitor_SMD:C_0805_2012Metric_Pad1.15x1.40mm_HandSolder
- removed C207: 22u, Capacitor_SMD:C_0805_2012Metric_Pad1.15x1.40mm_HandSolder
- removed C208: 18n, Capacitor_SMD:C_0805_2012Metric_Pad1.15x1.40mm_HandSolder
- removed C209: C11, Capacitor_SMD:C_0805_2012Metric_Pad1.15x1.40mm_HandSolder
- removed C210: C9, Capacitor_SMD:C_0805_2012Metric_Pad1.15x1.40mm_HandSolder
- removed C211: C10, Capacitor_SMD:C_0805_2012Metric_Pad1.15x1.40mm_HandSolder
- removed C212: 1n, Capacitor_SMD:C_0805_2012Metric_Pad1.15x1.40mm_HandSolder
- removed C213: C12, Capacitor_SMD:C_0805_2012Metric_Pad1.15x1.40mm_HandSolder
- removed C214: C8, Capacitor_SMD:C_0805_2012Metric_Pad1.15x1.40mm_HandSolder
- removed C215: C6, Capacitor_SMD:C_0805_2012Metric_Pad1.15x1.40mm_HandSolder
- removed C216: 47n, Capacitor_SMD:C_0805_2012Metric_Pad1.15x1.40mm_HandSolder
- removed C217: 10n, Capacitor_SMD:C_0805_2012Metric_Pad1.15x1.40mm_HandSolder
- removed C218: C7, Capacitor_SMD:C_0805_2012Metric_Pad1.15x1.40mm_HandSolder
- removed C219: C4, Capacitor_SMD:C_0805_2012Metric_Pad1.15x1.40mm_HandSolder
- removed C220, C221: 10u, Capacitor_SMD:C_1206_3216Metric_Pad1.42x1.75mm_HandSolder
- removed D201, D202: 1N1007, Diode_SMD:D_SOD-123
- removed D203, D204: D_Zener, Diode_SMD:D_MiniMELF
- removed D205, D206, D207, D208, D209: 1N4148, Diode_SMD:D_SOD-123
- removed the G*** at (94.5, 138.0)
- removed the G*** at (94.2, 138.5)
- removed H204: 2,2mm, MountingHole:MountingHole_2.2mm_M2_Pad_Via
- removed J201: In_Accent, Connector_Audio:Jack_3.5mm_Ledino_KB3SPRS_Horizontal
- removed J202: In Gate, AJ-Dropbox-Kicad:PJ301SM
- removed J203: Out Tom, AJ-Dropbox-Kicad:PJ301SM
- removed JP201: Jumper, Connector_PinHeader_2.54mm:PinHeader_1x02_P2.54mm_Vertical
- removed P201: Doepfer_Power_10pin, Connectors_IDC:IDC-Header_2x05_Pitch2.54mm_Straight
- removed Q201, Q202, Q203, Q204, Q206, Q207: MMBT2222A, Package_TO_SOT_SMD:SOT-23_Handsoldering
- removed Q205: MMBT2907A, Package_TO_SOT_SMD:SOT-23_Handsoldering
- removed R201, R206: 1M, Resistor_SMD:R_0805_2012Metric_Pad1.15x1.40mm_HandSolder
- removed R202, R220, R221, R228, R229, R233, R235, R238, R239, R242: 4k7, Resistor_SMD:R_0805_2012Metric_Pad1.15x1.40mm_HandSolder
- removed R203: 330K, Resistor_SMD:R_0805_2012Metric_Pad1.15x1.40mm_HandSolder
- removed R204: 100R, Resistor_SMD:R_0805_2012Metric_Pad1.15x1.40mm_HandSolder
- removed R205, R207, R232, R240, R241, R245, R250: 22k, Resistor_SMD:R_0805_2012Metric_Pad1.15x1.40mm_HandSolder
- removed R208: 300R, Resistor_SMD:R_0805_2012Metric_Pad1.15x1.40mm_HandSolder
- removed R209, R211: 1K, Resistor_SMD:R_0805_2012Metric_Pad1.15x1.40mm_HandSolder
- removed R210, R213: OPEN, Resistor_SMD:R_0805_2012Metric_Pad1.15x1.40mm_HandSolder
- removed R212: 0R, Resistor_SMD:R_0805_2012Metric_Pad1.15x1.40mm_HandSolder
- removed R214, R225: 1k, Resistor_SMD:R_0805_2012Metric_Pad1.15x1.40mm_HandSolder
- removed R215, R222: 470k, Resistor_SMD:R_0805_2012Metric_Pad1.15x1.40mm_HandSolder
- removed R216: 820k, Resistor_SMD:R_0805_2012Metric_Pad1.15x1.40mm_HandSolder
- removed R217, R223, R244, R249: 33k, Resistor_SMD:R_0805_2012Metric_Pad1.15x1.40mm_HandSolder
- removed R218, R219, R224, R234, R251, R252, R253, R254: 100k, Resistor_SMD:R_0805_2012Metric_Pad1.15x1.40mm_HandSolder
- removed R226: 15k, Resistor_SMD:R_0805_2012Metric_Pad1.15x1.40mm_HandSolder
- removed R227, R236, R237, R246: 10k, Resistor_SMD:R_0805_2012Metric_Pad1.15x1.40mm_HandSolder
- removed R230: R17, Resistor_SMD:R_0805_2012Metric_Pad1.15x1.40mm_HandSolder
- removed R231: R18, Resistor_SMD:R_0805_2012Metric_Pad1.15x1.40mm_HandSolder
- removed R243: 3k3, Resistor_SMD:R_0805_2012Metric_Pad1.15x1.40mm_HandSolder
- removed R247: 47k, Resistor_SMD:R_0805_2012Metric_Pad1.15x1.40mm_HandSolder
- removed R248: 2M2, Resistor_SMD:R_0805_2012Metric_Pad1.15x1.40mm_HandSolder
- removed RV201: 100K, Potentiometer_THT:Potentiometer_Bourns_3296W_Vertical
- removed RV202: 50K, Potentiometer_THT:Potentiometer_Bourns_3296W_Vertical
- removed RV203: 500R Tune, Potentiometer_THT:Potentiometer_Piher_T-16H_Single_Horizontal
- removed RV204: 1M Decay, Potentiometer_THT:Potentiometer_Piher_T-16H_Single_Horizontal
- removed RV205: 100k A Level, Potentiometer_THT:Potentiometer_Piher_T-16H_Single_Horizontal
- removed RV206: 100k A Reverb, Potentiometer_THT:Potentiometer_Piher_T-16H_Single_Horizontal
- removed SW201: Con/Tom, AJ-Dropbox-Kicad:SPDTx2
- removed TP201: WhiteNoise, TestPoint:TestPoint_Pad_1.5x1.5mm
- removed TP202: GND, TestPoint:TestPoint_THTPad_2.0x2.0mm_Drill1.0mm
- removed TP203: Coupling, TestPoint:TestPoint_Pad_1.5x1.5mm
- removed U201, U202, U203: TL072, AJ-Dropbox-Kicad:AJ_SO-8_5.3x6.2mm_P1.27mm
Routing:
- net +12V: track 359.5 -> 121.2 mm
- net GND: track 225.6 -> 17.8 mm, vias 145 -> 67
- net -12V: track 225.6 -> 68.3 mm
- net Net-(C210-Pad2): track 99.5 -> 0.00 mm, vias 2 -> 0
- net Net-(C209-Pad2): track 56.0 -> 0.00 mm, vias 2 -> 0
- net Net-(C218-Pad1): track 54.1 -> 0.00 mm, vias 4 -> 0
- net Net-(C212-Pad2): track 52.9 -> 0.00 mm, vias 4 -> 0
- net Net-(C212-Pad1): track 48.4 -> 0.00 mm, vias 5 -> 0
- net /KicadJE_AteOhAte2/PNP_E: track 42.9 -> 0.00 mm
- net /KicadJE_AteOhAte2/WhiteNoise: track 42.5 -> 0.00 mm, vias 3 -> 0
- net Net-(R217-Pad1): track 41.9 -> 0.00 mm
- net /KicadJE_AteOhAte2/Coupling: track 41.4 -> 0.00 mm, vias 5 -> 0
- net InAccent: track 35.5 -> 0.00 mm
- net Net-(C213-Pad1): track 33.7 -> 0.00 mm
- net Net-(D205-Pad1): track 33.3 -> 0.00 mm
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Other:
- outline, holes or cut-outs redrawn
- board text removed: "DRUM_Ate0Ate_Tom_1 Rev A - 25/09-2019 Johansen Engineering"
- board text removed: "Reg noise to 130mV"

Commit message: SCH incl AC driver
Other:
- board size 100 x 100 mm -> 100 x 91.8 mm
Changed lines of the file:
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@@
   (general
     (thickness 1.6)
-    (drawings 42)
+    (drawings 46)
     (tracks 448)
     (zones 0)
@@
     (38 B.Mask user)
     (39 F.Mask user)
-    (40 Dwgs.User user)
+    (40 Dwgs.User user hide)
     (41 Cmts.User user)
     (42 Eco1.User user)
@@
     )
   )
+  (gr_line (start 99 138.5) (end 100 138.5) (layer Edge.Cuts) (width 1))
+  (gr_line (start 99 82.25) (end 99 138.5) (layer Edge.Cuts) (width 1))
+  (gr_line (start 100 82.25) (end 99 82.25) (layer Edge.Cuts) (width 1))
+  (gr_line (start 100 138.5) (end 100 82.25) (layer Edge.Cuts) (width 1))
   (gr_text Input (at 145.5 108) (layer F.SilkS)
     (effects (font (size 0.8 0.8) (thickness 0.1)) (justify left))
@@
   (gr_line (start 50 119.9) (end 150 119.9) (layer Dwgs.User) (width 0.15))
   (gr_line (start 50 143.9) (end 150 143.9) (layer Dwgs.User) (width 0.15))
-  (gr_line (start 50 150) (end 50 50) (layer Edge.Cuts) (width 0.05))
+  (gr_line (start 50 145.5) (end 50 53.75) (layer Edge.Cuts) (width 0.05))
   (gr_line (start 150 145.5) (end 50 145.5) (layer Edge.Cuts) (width 0.05))
   (gr_line (start 150 53.75) (end 150 145.5) (layer Edge.Cuts) (width 0.05))

Commit message: hopefully it works
Parts:
- added C101: 470u, Capacitor_THT:CP_Radial_D13.0mm_P5.00mm, F.Cu at (81.0, 64.0)
- added C102: 470u, Capacitor_THT:CP_Radial_D13.0mm_P5.00mm, F.Cu at (81.0, 79.0)
- added C103: 100n, Capacitor_SMD:C_0805_2012Metric_Pad1.15x1.40mm_HandSolder, F.Cu at (72.2, 72.0)
- added C104: 100n, Capacitor_SMD:C_0805_2012Metric_Pad1.15x1.40mm_HandSolder, F.Cu at (72.2, 76.0)
- added C105: 100n, Capacitor_SMD:C_0805_2012Metric_Pad1.15x1.40mm_HandSolder, F.Cu at (87.0, 99.2)
- added C106: 100n, Capacitor_SMD:C_0805_2012Metric_Pad1.15x1.40mm_HandSolder, F.Cu at (87.5, 115.5)
- added C107: 100n, Capacitor_SMD:C_0805_2012Metric_Pad1.15x1.40mm_HandSolder, F.Cu at (64.2, 103.2)
- added C108: 100n, Capacitor_SMD:C_0805_2012Metric_Pad1.15x1.40mm_HandSolder, F.Cu at (80.5, 127.5)
- added C109: 100n, Capacitor_SMD:C_0805_2012Metric_Pad1.15x1.40mm_HandSolder, F.Cu at (64.8, 126.8)
- added C110: 100n, Capacitor_SMD:C_0805_2012Metric_Pad1.15x1.40mm_HandSolder, F.Cu at (80.5, 132.2)
- added C111: 100n, Capacitor_SMD:C_0805_2012Metric_Pad1.15x1.40mm_HandSolder, F.Cu at (64.2, 111.8)
- added C112: 100n, Capacitor_SMD:C_0805_2012Metric_Pad1.15x1.40mm_HandSolder, F.Cu at (65.0, 134.5)
- added C302: 100u, Capacitor_SMD:CP_Elec_8x6.5, F.Cu at (130.0, 69.5)
- added C316: 100u, Capacitor_SMD:CP_Elec_8x6.5, F.Cu at (145.0, 69.5)
- added C344: 22u, Capacitor_THT:CP_Radial_D8.0mm_P3.50mm, F.Cu at (130.5, 132.5)
- added D101: DF08M, Diode_THT:Diode_Bridge_DIP-4_W7.62mm_P5.08mm, F.Cu at (68.0, 70.2)
- added D102: LED, LED_THT:LED_D3.0mm, F.Cu at (94.8, 88.8)
- added D103: LED, LED_THT:LED_D3.0mm, F.Cu at (82.2, 105.8)
- added D104: LED, LED_THT:LED_D3.0mm, F.Cu at (82.2, 111.8)
- added H301: 2,5mm, MountingHole:MountingHole_2.5mm_Pad_Via, F.Cu at (89.2, 58.5)
- added H302: 2,2mm, MountingHole:MountingHole_2.2mm_M2_Pad_Via, F.Cu at (94.8, 96.8)
- added H302: 2,2mm, MountingHole:MountingHole_2.2mm_M2_Pad_Via, F.Cu at (54.5, 96.8)
- added H302: 2,2mm, MountingHole:MountingHole_2.2mm_M2_Pad_Via, F.Cu at (54.5, 141.5)
- added H303: 2,5mm, MountingHole:MountingHole_2.5mm_Pad_Via, F.Cu at (54.5, 58.2)
- added H304: 2,2mm, MountingHole:MountingHole_2.2mm_M2_Pad_Via, F.Cu at (89.3, 141.5)
- added J101: Conn_01x03, TerminalBlock:TerminalBlock_bornier-3_P5.08mm, F.Cu at (94.0, 79.5)
- added J102: Conn_01x03, TerminalBlock:TerminalBlock_bornier-3_P5.08mm, F.Cu at (54.2, 69.0)
- added J103: Conn_01x03, TerminalBlock:TerminalBlock_bornier-3_P5.08mm, F.Cu at (94.2, 112.8)
- added J104: Conn_01x03, TerminalBlock:TerminalBlock_bornier-3_P5.08mm, F.Cu at (94.2, 135.0)
- added J301: PJRAS2X2S01AUX, AJ:PJRAS2X2S01AUX_RCA, F.Cu at (141.0, 123.0)
- added Q101: BD139, Package_TO_SOT_THT:TO-126-3_Vertical, F.Cu at (56.5, 106.2)
- added Q102: BD140, Package_TO_SOT_THT:TO-126-3_Vertical, F.Cu at (56.5, 115.2)
- added Q103: MMBT2222A, Package_TO_SOT_SMD:SOT-23_Handsoldering, F.Cu at (59.8, 127.0)
- added Q104: BD139, Package_TO_SOT_THT:TO-126-3_Vertical, F.Cu at (54.0, 128.0)
- added Q105: MMBT2907A, Package_TO_SOT_SMD:SOT-23_Handsoldering, F.Cu at (59.8, 132.2)
- added Q106: BD140, Package_TO_SOT_THT:TO-126-3_Vertical, F.Cu at (54.0, 136.8)
- added R101: 1R1, Resistor_SMD:R_0805_2012Metric_Pad1.15x1.40mm_HandSolder, F.Cu at (72.0, 64.0)
- added R102: 12k, Resistor_SMD:R_0805_2012Metric_Pad1.15x1.40mm_HandSolder, B.Cu at (95.0, 56.0)
- added R103: 1R1, Resistor_SMD:R_0805_2012Metric_Pad1.15x1.40mm_HandSolder, F.Cu at (72.0, 84.0)
- added R104: 22R, Resistor_THT:R_Axial_DIN0309_L9.0mm_D3.2mm_P15.24mm_Horizontal, F.Cu at (75.2, 99.5)
- added R105: 10k, Resistor_SMD:R_0805_2012Metric_Pad1.15x1.40mm_HandSolder, F.Cu at (82.5, 99.2)
- added R106: 1k, Resistor_SMD:R_0805_2012Metric_Pad1.15x1.40mm_HandSolder, F.Cu at (64.2, 107.8)
- added R107: 10k, Resistor_SMD:R_0805_2012Metric_Pad1.15x1.40mm_HandSolder, F.Cu at (82.2, 115.5)
- added R108: 22R, Resistor_THT:R_Axial_DIN0309_L9.0mm_D3.2mm_P15.24mm_Horizontal, F.Cu at (75.2, 115.8)
- added R109: 22R, Resistor_THT:R_Axial_DIN0309_L9.0mm_D3.2mm_P15.24mm_Horizontal, F.Cu at (77.2, 122.0)
- added R110: 22k, Resistor_SMD:R_0805_2012Metric_Pad1.15x1.40mm_HandSolder, F.Cu at (88.7, 127.5)
- added R111: 18k, Resistor_SMD:R_0805_2012Metric_Pad1.15x1.40mm_HandSolder, F.Cu at (84.5, 127.5)
- added R112: 1k, Resistor_SMD:R_0805_2012Metric_Pad1.15x1.40mm_HandSolder, F.Cu at (64.8, 130.5)
- added R113: 22k, Resistor_SMD:R_0805_2012Metric_Pad1.15x1.40mm_HandSolder, F.Cu at (88.7, 132.2)
- added R114: 18k, Resistor_SMD:R_0805_2012Metric_Pad1.15x1.40mm_HandSolder, F.Cu at (84.5, 132.2)
- added R115: 22R, Resistor_THT:R_Axial_DIN0309_L9.0mm_D3.2mm_P15.24mm_Horizontal, F.Cu at (76.5, 140.2)
- added U101: TL071, Package_DIP:DIP-8_W7.62mm_LongPads, F.Cu at (69.0, 111.2)
- added U102: TL071, Package_DIP:DIP-8_W7.62mm_LongPads, F.Cu at (69.0, 134.2)
- moved J302 0.25 mm to (105.0, 79.8)
Connections:
- F301 pad 1: /KicadJE_AteOhAte3/+PSU -> (no net)
- F302 pad 2: /KicadJE_AteOhAte3/-PSU -> (no net)
- J302 pad 1: /KicadJE_AteOhAte3/-PSU -> /-PSU
- J302 pad 2: (no net) -> GND
- J302 pad 3: /KicadJE_AteOhAte3/+PSU -> /+PSU
Routing:
- net GND: track 17.8 -> 351.8 mm, vias 67 -> 103
- net /+PSU: track 0.00 -> 190.3 mm
- net /-PSU: track 0.00 -> 188.9 mm
- net Net-(C109-Pad1): track 0.00 -> 42.2 mm
- net Net-(D102-Pad2): track 0.00 -> 38.4 mm
- net Net-(C107-Pad1): track 0.00 -> 34.8 mm
- net Net-(C105-Pad1): track 0.00 -> 28.3 mm
- net Net-(C108-Pad1): track 0.00 -> 25.6 mm
- net /BR-: track 0.00 -> 19.6 mm
- net Net-(Q105-Pad3): track 0.00 -> 16.1 mm
- net /AC3: track 0.00 -> 14.3 mm
- net /AC1: track 0.00 -> 13.6 mm
- net Net-(Q103-Pad3): track 0.00 -> 13.2 mm
- net /BR+: track 0.00 -> 12.0 mm
- net Net-(R106-Pad2): track 0.00 -> 10.8 mm
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Other:
- board text added: "- +"
- board text added: "AC"
- board text added: "AC 12"

Commit message: DRC
Parts:
- removed the J301 at (141.0, 123.0)
Routing:
- net Out_L: track 39.9 -> 56.0 mm
